File: kicad/gps.kicad_pcb (KiCad board)
At the start: 4 copper layers, 84.1 x 61.7 mm, 66 parts, among them J1 Bus_PCI_Express_x1, J2 USB_C_Receptacle_USB2.0_16P, J3 Conn_01x03, J4 USB_C_Receptacle_USB2.0_16P, J5 Conn_01x02_Pin, Q1 IRLML6344, U2 W25Q128JVP, U3 MCP25625T-E/ML, U4 RP2040, U5 NEO-M9N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

Commit message: Generate Fabrication Files
Routing:
- net +3.3V: track 190.7 -> 192.0 mm, vias 12 -> 15
- net /QSPI_SS: track 42.1 -> 42.9 mm
- net +5V: vias 1 -> 4
Changed lines of the file:
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@@
 	)
 	(via
-		(at 152.4 118.618)
+		(at 152.43 119.27)
 		(size 0.4)
 		(drill 0.3)
@@
 	)
 	(segment
+		(start 166.008554 106.1725)
+		(end 174.6125 106.1725)
+		(width 0.15)
+		(layer "F.Cu")
+		(net 19)
+	)
+	(segment
+		(start 168.04006 118.02994)
+		(end 151.46606 118.02994)
+		(width 0.15)
+		(layer "F.Cu")
+		(net 19)
+	)
+	(segment
+		(start 174.6125 106.1725)
+		(end 175.92 107.48)
+		(width 0.15)
+		(layer "F.Cu")
+		(net 19)
+	)
+	(segment
+		(start 165.7425 105.906446)
+		(end 166.008554 106.1725)
+		(width 0.15)
+		(layer "F.Cu")
+		(net 19)
+	)
+	(segment
+		(start 175.92 107.48)
+		(end 175.92 110.3)
+		(width 0.15)
+		(layer "F.Cu")
+		(net 19)
+	)
+	(segment
 		(start 151.46606 118.02994)
 		(end 151.005 118.491)
@@
 	)
 	(segment
-		(start 166.008554 106.1725)
-		(end 174.6125 106.1725)
-		(width 0.15)
-		(layer "F.Cu")
-		(net 19)
-	)
-	(segment
-		(start 174.6125 106.1725)
-		(end 175.92 107.48)
-		(width 0.15)
-		(layer "F.Cu")
-		(net 19)
-	)
-	(segment
-		(start 165.7425 105.906446)
-		(end 166.008554 106.1725)
-		(width 0.15)
-		(layer "F.Cu")
-		(net 19)
-	)
-	(segment
-		(start 168.42054 118.02994)
-		(end 151.46606 118.02994)
-		(width 0.15)
-		(layer "F.Cu")
-		(net 19)
-	)
-	(segment
-		(start 175.92 107.48)
-		(end 175.92 110.3)
-		(width 0.15)
-		(layer "F.Cu")
-		(net 19)
-	)
-	(segment
 		(start 175.92 110.3)
 		(end 173.8925 112.3275)
+		(width 0.15)
+		(layer "F.Cu")
+		(net 19)
+	)
+	(segment
+		(start 168.865 117.205)
+		(end 168.04006 118.02994)
 		(width 0.15)
 		(layer "F.Cu")
@@
 	)
 	(segment
+		(start 145.913 64.138595)
+		(end 145.913 68.090384)
+		(width 0.3)
+		(layer "F.Cu")
+		(net 26)
+	)
+	(segment
 		(start 162.9425 96.5525)
 		(end 162.7925 96.4025)
@@
 	)
 	(segment
-		(start 145.913 64.138595)
-		(end 145.913 68.082)
-		(width 0.3)
-		(locked yes)
-		(layer "F.Cu")
-		(net 26)
-	)
-	(segment
 		(start 158.691353 100.985)
 		(end 157.907179 100.200826)
@@
 	)
 	(segment
-		(start 145.913 68.082)
-		(end 145.913 68.090384)
-		(width 0.3)
-		(layer "F.Cu")
-		(net 26)
-	)
-	(segment
 		(start 118.39 107.86)
 		(end 118.39 114.048598)
@@
 		(start 139.869405 74.249578)
 		(end 138.898299 75.220684)
+		(width 0.3)
+		(layer "F.Cu")
+		(net 26)
+	)
+	(segment
+		(start 145.913 68.090384)
+		(end 140.408382 73.595002)
 		(width 0.3)
 		(layer "F.Cu")
@@
 	)
 	(segment
-		(start 145.913 68.090384)
-		(end 140.408382 73.595002)
-		(width 0.3)
-		(layer "F.Cu")
-		(net 26)
-	)
-	(segment
 		(start 118.39 114.048598)
 		(end 119.6 115.258598)
@@
 	)
 	(via
+		(at 144.91 65.26)
+		(size 0.4)
+		(drill 0.3)
+		(layers "F.Cu" "B.Cu")
+		(net 26)
+	)
+	(via
 		(at 144.478301 80.416276)
 		(size 0.4)
@@
 	)
 	(via
+		(at 146.91 65.27)
+		(size 0.4)
+		(drill 0.3)
+		(layers "F.Cu" "B.Cu")
+		(net 26)
+	)
+	(via
 		(at 157.0425 105.1725)
 		(size 0.4)
@@
 		(layers "F.Cu" "B.Cu")
 		(free yes)
+		(net 26)
+	)
+	(via
+		(at 145.91 65.27)
+		(size 0.4)
+		(drill 0.3)
+		(layers "F.Cu" "B.Cu")
 		(net 26)
 	)
@@
 	)
 	(segment
+		(start 140.12 73.9)
+		(end 128 73.9)
+		(width 0.3)
+		(layer "B.Cu")
+		(net 26)
+	)
+	(segment
 		(start 145.744789 79.639788)
 		(end 146.459375 78.925202)
@@
 	)
 	(segment
-		(start 137.951595 73.9)
-		(end 145.913 65.938595)
-		(width 0.3)
-		(layer "B.Cu")
-		(net 26)
-	)
-	(segment
 		(start 167.2925 107.4225)
 		(end 166.5425 106.6725)
@@
 	)
 	(segment
+		(start 145.913 64.138595)
+		(end 145.913 68.107)
+		(width 0.3)
+		(layer "B.Cu")
+		(net 26)
+	)
+	(segment
 		(start 146.459375 78.925202)
 		(end 146.459375 78.939325)
@@
 	)
 	(segment
-		(start 118.39 83.51)
-		(end 128 73.9)
-		(width 0.3)
-		(layer "B.Cu")
-		(net 26)
-	)
-	(segment
 		(start 146.129375 75.979325)
 		(end 146.459375 76.309325)
@@
 	)
 	(segment
-		(start 128 73.9)
-		(end 137.951595 73.9)
-		(width 0.3)
-		(layer "B.Cu")
-		(net 26)
-	)
-	(segment
 		(start 166.000501 104.943476)
 		(end 166.500501 105.443476)
@@
 		(end 166.5425 105.4225)
 		(width 0.4)
-		(layer "B.Cu")
-		(net 26)
-	)
-	(segment
-		(start 145.913 65.938595)
-		(end 145.913 64.138595)
-		(width 0.3)
-		(layer "B.Cu")
-		(net 26)
-	)
-	(segment
-		(start 118.39 107.86)
-		(end 118.39 83.51)
-		(width 0.3)
 		(layer "B.Cu")
 		(net 26)
@@
 	)
 	(segment
+		(start 118.39 83.51)
+		(end 118.39 107.86)
+		(width 0.3)
+		(layer "B.Cu")
+		(net 26)
+	)
+	(segment
+		(start 128 73.9)
+		(end 118.39 83.51)
+		(width 0.3)
+		(layer "B.Cu")
+		(net 26)
+	)
+	(segment
 		(start 145.881001 66.092976)
 		(end 145.881001 64.144571)
@@
 	)
 	(segment
+		(start 145.913 68.107)
+		(end 140.12 73.9)
+		(width 0.3)
+		(layer "B.Cu")
+		(net 26)
+	)
+	(segment
 		(start 144.038999 81.242298)
 		(end 144.533999 81.737298)
@@
 	)
 	(via
+		(at 151.92 65.26)
+		(size 0.4)
+		(drill 0.3)
+		(layers "F.Cu" "B.Cu")
+		(net 29)
+	)
+	(via
+		(at 150.94 65.27)
+		(size 0.4)
+		(drill 0.3)
+		(layers "F.Cu" "B.Cu")
+		(net 29)
+	)
+	(via
 		(at 135.0103 79.689324)
 		(size 0.4)
 		(drill 0.3)
+		(layers "F.Cu" "B.Cu")
+		(net 29)
+	)
+	(via
+		(at 149.9 65.27)
+		(size 0.4)
+		(drill 0.3)

Commit message: Final Commit before 0.2.0 Order
Parts:
- RF1: value BWSMA-KE-P001 -> BWSMA-KWE-Z001
Changed lines of the file:
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@@
 			)
 		)
+		(property ki_fp_filters "Connector*:*_1x??_*")
+		(sheetname "/")
+		(sheetfile "gps.kicad_sch")
 		(attr through_hole dnp)
 		(fp_line
@@
 			)
 		)
+		(property ki_fp_filters "R_*")
+		(sheetname "/")
+		(sheetfile "gps.kicad_sch")
 		(attr smd)
 		(fp_line
@@
 			)
 		)
-		(property "Value" "BWSMA-KE-P001"
+		(property "Value" "BWSMA-KWE-Z001"
 			(at 0 0.210027 270)
 			(unlocked yes)
@@
 			)
 		)
-		(property "JLC Link" "https://jlcpcb.com/partdetail/C496550"
+		(property "JLC Link" "https://jlcpcb.com/partdetail/C496551"
 			(at 0 0 270)
 			(unlocked yes)
@@
 			)
 		)
-		(property "LCSC Part #" "C496550"
+		(property "LCSC Part #" "C496551"
 			(at 0 0 270)
 			(unlocked yes)
@@
 			)
 		)
-		(property "Manufacturer Part Number" "BWSMA-KE-P001"
+		(property "Manufacturer Part Number" "BWSMA-KWE-Z001"
 			(at 0 0 270)
 			(unlocked yes)
