File: kicad/gps.kicad_sch (KiCad schematic)
At the start: 71 parts, among them J1 Bus_PCI_Express_x1, J2 USB_C_Receptacle_USB2.0_16P, J3 Conn_01x03, J4 USB_C_Receptacle_USB2.0_16P, J5 Conn_01x02_Pin, Q2 BSS84, U1 SI1016X-T1-GE3, U2 W25Q128JVP, U3 MCP25625T-E/ML, U4 RP2040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

Commit message: Major updates
Parts:
- removed BAT: JUMPER-SMT_2_NC_TRACE_SILK, GPSLIB:SMT-JUMPER_2_NC_TRACE_SILK, symbol SparkFun u-blox GNSS MAX-M10S-eagle-import:JUMPER-SMT_2_NC_TRACE_SILK
- removed Q2: BSS84, Package_TO_SOT_SMD:SOT-23, symbol Transistor_FET:BSS84
- removed R18: 1k, Resistor_SMD:R_0402_1005Metric, symbol Device:R
- added C24, C25: 1u, Capacitor_SMD:C_0402_1005Metric, symbol Device:C
- added C26, C27: 100n, Capacitor_SMD:C_0402_1005Metric, symbol Device:C
- added R6: 10k, Resistor_SMD:R_0402_1005Metric, symbol Device:R
- added U7: RT9013-33GB, GPSLIB:SOT-23-5_RIT_LDO, symbol gpsmodule:RT9013-33GB
- added U8: TPS2115APWR, GPSLIB:PW8, symbol gpsmodule:TPS2115APWR
- added VCC_RF: JUMPER-SMT_2_NC_TRACE_SILK, GPSLIB:SMT-JUMPER_2_NC_TRACE_SILK, symbol SparkFun u-blox GNSS MAX-M10S-eagle-import:JUMPER-SMT_2_NC_TRACE_SILK
- R10: value 10k -> 100k; Basic? (none) -> Yes; Current Draw (none) -> N/A (passive component); Height (none) -> Approximately 0.4 mm; Info (none) -> -55℃~+155℃ 100kΩ 50V 62.5mW Thick Film Resistor ±1% ±100ppm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; JLC Link https://jlcpcb.com/partdetail/26487-0402WGF1002TCE/C25744 -> https://jlcpcb.com/partdetail/26484-0402WGF1003TCE/C25741; LCSC Part # C25744 -> C25741; Manufacturer Name (none) -> UNI-ROYAL (Uniroyal Elec); Manufacturer Part Number (none) -> 0402WGF1003TCE; Mouser Part Number (none) -> Not listed; Mouser Price/Stock (none) -> Not listed; Notes (none) -> Suitable for general-purpose surface-mount applications; Ro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; Price (none) -> Approximately C$0.0005 per unit (bulk pricing available); basic? yes -> (none); info 10k ohm -> (none); price C$0.0007 -> (none)
- R13: value 10k -> 499R; Basic? (none) -> Yes; Current Draw (none) -> N/A (passive component); Height (none) -> Approximately 0.4 mm; Info (none) -> -55℃~+155℃ 100kΩ 50V 62.5mW Thick Film Resistor ±1% ±100ppm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; JLC Link https://jlcpcb.com/partdetail/26487-0402WGF1002TCE/C25744 -> https://jlcpcb.com/partdetail/4532-0402WGF4990TCE/C4125; LCSC Part # C25744 -> C4125; Manufacturer Name (none) -> UNI-ROYAL (Uniroyal Elec); Manufacturer Part Number (none) -> 0402WGF4990TCE; Mouser Part Number (none) -> Not listed; Mouser Price/Stock (none) -> Not listed; Notes (none) -> Suitable for general-purpose surface-mount applications; Ro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; Price (none) -> Approximately C$0.0005 per unit (bulk pricing available); basic? yes -> (none); info 10k ohm -> (none); price C$0.0007 -> (none)
- R9: value 3.3k -> 75R; footprint Resistor_SMD:R_0402_1005Metric -> Resistor_SMD:R_0805_2012Metric; JLC Link https://jlcpcb.com/partdetail/26679-0402WGJ0332TCE/C25936 -> https://jlcpcb.com/partdetail/18508-0805W8F750JT5E/C17820; LCSC Part # C25936 -> C17820; Manufacturer_Name (none) -> UNI-ROYAL(Uniroyal Elec); Manufacturer_Part_Number (none) -> 0805W8F750JT5E; info 3.3k ohm -> 120 ohm
- U5: footprint GPSLIB:XCVR_NEO-M9N-00B -> RF_GPS:ublox_NEO; Basic? No -> (none); Current Draw ~29 mA (continuous tracking) -> (none); Height 2.4 mm -> (none); Info GNSS Receiver Module (GPS, GLONASS, Galileo, BeiDou) -> (none); JLC Link https://jlcpcb.com/partdetail/ublox-NEO_M9N00B/C5119087 -> (none); LCSC Part # C5119087 -> (none); Manufacturer Name u-blox -> (none); Manufacturer Part Number NEO-M9N-00B-00 -> (none); Mouser Part Number 377-NEO-M9N-00B-00 -> (none); Mouser Price/Stock C$19.60 / In Stock -> (none); Notes Supports concurrent GNSS, UART/SPI/I2C, high update rate (u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 -> (none); Price C$15.1029 -> (none)
- U6: Basic Part? (none) -> Yes; Current Draw (none) -> Output sink current max: 32 mA; Info (none) -> Dual non-inverting open-drain buffer; SOT-363; CMOS; ROHS; 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; JLC Link (none) -> https://jlcpcb.com/partdetail/onsemi-NC7WZ07P6X/C95342; LCSC Part # (none) -> C95342; MFR.Part # (none) -> NC7WZ07P6X; Manufacturer (none) -> onsemi; Price (none) -> C$0.0850 (1+), down to C$0.0418 (9000+)
Connections:
- net USB_SENSE is gone; now on net LDO_OUT: U5.7 (VDD_USB)
- net +3.3V: now also C26.1, U8.8 (IN1); no longer U5.23 (VCC)
- net BACKUP: now also R9.2
- net BIAS_T: now also U6.1 (A1), VCC_RF.1
- net GND: now also R13.2, C24.1, C25.1, C26.2, C27.2, U7.2 (GND), U8.3 (D1), U8.5 (GND)
- net VCC_RF: now also VCC_RF.2
- net LDO_OUT: now reaches R10.1
- net LDO_OUT: now also C25.2, C27.1, U7.5 (VOUT), U8.6 (IN2); no longer R13.2
- net at D2.C: now also R9.1; no longer R9.2
- net ANT_SWITCH_N: now reaches U5.16 (ANT_SWITCH_N)
- net ANT_SWITCH_N: now also U6.6 (Y1)
- net V_USB renamed GPS_USB_PWR
- net GPS_USB_PWR: now also C24.2, R6.1, U7.1 (VIN); no longer R13.1
- new net: R13.1, U8.4 (ILIM)
- new net: R6.2, U7.3 (EN)
- new net MUX_OUT: U5.23 (VCC), U8.7 (OUT)
- no-connect marks 47 -> 52
Other:
- note added: "V=3.3V, R=75, I(max)=44mA Usable voltage range: 1.65V - 3.60V 95% of 3.3v in 105.6 sec"
- moved on the sheet: R5, R9, U1, U6
